Commit message: Completed Task B.001

File: nuturtle_description/urdf/diff_drive.urdf.xacro (robot description, xacro)
@@ -57,5 +57,5 @@
         <box size="${chassis_length} ${chassis_width} ${chassis_thickness}" />
       </geometry>
-      <origin rpy="0 0 0" xyz="${chassis_length/2 - wheel_radius} 0 ${wheel_radius}"/>
+      <origin rpy="0 0 0" xyz="${base_shift} 0 ${wheel_radius}"/>
       <material name="green_mat">
         <color rgba="0 1 0 1" />

Commit message: Successfully running all code for Task F.007

File: nuturtle_description/urdf/diff_drive.urdf.xacro (robot description, xacro)
@@ -10,5 +10,5 @@
   <xacro:property name="chassis_thickness" value="${props['chassis_thickness']}"/>
   <xacro:property name="chassis_width" value="${(wheel_base - wheel_width)}"/>
-  <xacro:property name="castor_radius" value="${((wheel_radius - (chassis_thickness/2))/2)}"/>
+  <xacro:property name="castor_radius" value="${(wheel_radius/2)}"/>
   <xacro:property name="base_shift" value="${chassis_length/2 - wheel_radius}"/>
   <!-- Macro to create wheels -->
@@ -42,9 +42,10 @@
           <color rgba=".9 .9 .9 .95" />
         </material>
-        <origin rpy="0 0 0" xyz="0 0 0"/>
+        <origin rpy="0 0 0" xyz="0 0 ${castor_radius}"/>
       </visual>
     </link>
+    <!--  -->
     <joint name="${caster_side}_castor_joint" type="fixed">
-      <origin xyz="${base_shift + (chassis_length/2 - castor_radius)} 0 ${castor_radius}" rpy="0 0 0" />
+      <origin xyz="${base_shift + (chassis_length/2 - castor_radius)} 0 0" rpy="0 0 0" />
       <parent link="base_link"/>
       <child link="caster_${caster_side}" />
@@ -57,5 +58,5 @@
         <box size="${chassis_length} ${chassis_width} ${chassis_thickness}" />
       </geometry>
-      <origin rpy="0 0 0" xyz="${base_shift} 0 ${wheel_radius}"/>
+      <origin rpy="0 0 0" xyz="${base_shift} 0 ${wheel_radius + chassis_thickness/2}"/>
       <material name="green_mat">
         <color rgba="0 1 0 1" />

Commit message: Completed Task A.006

File: nuturtle_description/urdf/diff_drive.urdf.xacro (robot description, xacro)
@@ -9,7 +9,8 @@
   <xacro:property name="chassis_length" value="${props['chassis_length']}"/>
   <xacro:property name="chassis_thickness" value="${props['chassis_thickness']}"/>
+  <xacro:property name="wheel_axle_offset" value="${props['wheel_axle_offset']}"/>
   <xacro:property name="chassis_width" value="${(wheel_base - wheel_width)}"/>
-  <xacro:property name="castor_radius" value="${(wheel_radius/2)}"/>
   <xacro:property name="base_shift" value="${chassis_length/2 - wheel_radius}"/>
+  <xacro:property name="castor_radius" value="${wheel_axle_offset/2}"/>
   <!-- Macro to create wheels -->
   <xacro:macro name="wheel_temp" params="wheel_side offset">
@@ -24,7 +25,16 @@
         <origin rpy="${pi/2} 0 0" xyz="0 ${offset * (wheel_width/2)} 0"/>
       </visual>
+      <inertial>
+        <mass value="0.1"/>
+        <inertia ixx="${(1/12)*0.1*(3*wheel_radius**2+wheel_width**2)}" iyy="${.5*0.1*wheel_radius**2}" izz="${(1/12)*0.1*(3*wheel_radius**2+wheel_width**2)}" ixy="0" ixz="0" iyz="0"/>
+      </inertial>
+      <collision>
+        <geometry>
+            <cylinder length="${wheel_width}" radius="${wheel_radius}" />
+        </geometry>
+      </collision>
     </link>
     <joint name="${wheel_side}_wheel_axel" type="continuous">
-      <origin xyz="${base_shift-.25*chassis_length} ${offset * (chassis_width/2)} ${wheel_radius}" rpy="0 0 0" />
+      <origin xyz="${base_shift-.25*chassis_length} ${offset * (chassis_width/2)} ${wheel_axle_offset}" rpy="0 0 0" />
       <parent link="base_link"/>
       <child link="wheel_${wheel_side}" />
@@ -44,4 +54,9 @@
         <origin rpy="0 0 0" xyz="0 0 ${castor_radius}"/>
       </visual>
+      <collision>
+        <geometry>
+            <sphere radius="${castor_radius}" />
+        </geometry>
+      </collision>
     </link>
     <!--  -->
@@ -52,16 +67,33 @@
     </joint>
   </xacro:macro>
+  <link name="base_link">
+    <origin rpy="0 0 0" xyz="${base_shift} 0 0"/>
+  </link>
   <!-- The body of the robot-->
-  <link name="base_link" >
+  <link name="robot_body" >
     <visual>
       <geometry>
         <box size="${chassis_length} ${chassis_width} ${chassis_thickness}" />
       </geometry>
-      <origin rpy="0 0 0" xyz="${base_shift} 0 ${wheel_radius + chassis_thickness/2}"/>
+      <origin rpy="0 0 0" xyz="0 0 0"/>
       <material name="green_mat">
         <color rgba="0 1 0 1" />
       </material>
     </visual>
+    <inertial>
+      <mass value="1.0"/>
+      <inertia ixx="${(1/12)*(chassis_thickness**2 + chassis_width**2)}" iyy="${(1/12)*(chassis_thickness**2 + chassis_length**2)}" izz="${(1/12)*(chassis_length**2 + chassis_width**2)}" ixy="0" ixz="0" iyz="0"/>
+    </inertial>
+    <collision>
+      <geometry>
+        <box size="${chassis_length} ${chassis_width} ${chassis_thickness}" />
+      </geometry>
+    </collision>
   </link>
+  <joint name="base_body" type="fixed">
+    <origin xyz="${base_shift} 0 ${wheel_axle_offset + chassis_thickness/2}" rpy="0 0 0" />
+    <parent link="base_link"/>
+    <child link="robot_body"/>
+  </joint>
   <!-- Wheel Creation -->
   <xacro:wheel_temp wheel_side="left" offset="1"/>

Commit message: Completed Task G.001

File: nuturtle_description/urdf/diff_drive.urdf.xacro (robot description, xacro)
@@ -26,8 +26,10 @@
       </visual>
       <inertial>
+        <origin xyz="0 ${offset * wheel_width/2} 0"/>
         <mass value="0.1"/>
         <inertia ixx="${(1/12)*0.1*(3*wheel_radius**2+wheel_width**2)}" iyy="${.5*0.1*wheel_radius**2}" izz="${(1/12)*0.1*(3*wheel_radius**2+wheel_width**2)}" ixy="0" ixz="0" iyz="0"/>
       </inertial>
       <collision>
+        <origin rpy="${pi/2} 0 0" xyz="0 ${offset * (wheel_width/2)} 0"/>
         <geometry>
             <cylinder length="${wheel_width}" radius="${wheel_radius}" />
@@ -36,5 +38,5 @@
     </link>
     <joint name="${wheel_side}_wheel_axel" type="continuous">
-      <origin xyz="${base_shift-.25*chassis_length} ${offset * (chassis_width/2)} ${wheel_axle_offset}" rpy="0 0 0" />
+      <origin xyz="${base_shift-.25*chassis_length} ${offset * (chassis_width/2)} ${wheel_radius}" rpy="0 0 0" />
       <parent link="base_link"/>
       <child link="wheel_${wheel_side}" />
@@ -43,5 +45,5 @@
   </xacro:macro>
   <!-- Macro to create casters -->
-  <xacro:macro name="caster_temp" params="caster_side offset">
+  <xacro:macro name="caster_temp" params="caster_side">
     <link name="caster_${caster_side}">
       <visual>
@@ -55,4 +57,5 @@
       </visual>
       <collision>
+        <origin rpy="0 0 0" xyz="0 0 ${castor_radius}"/>
         <geometry>
             <sphere radius="${castor_radius}" />
@@ -76,5 +79,5 @@
         <box size="${chassis_length} ${chassis_width} ${chassis_thickness}" />
       </geometry>
-      <origin rpy="0 0 0" xyz="0 0 0"/>
+      <origin rpy="0 0 0" xyz="0 0 ${wheel_axle_offset + chassis_thickness/2}"/>
       <material name="green_mat">
         <color rgba="0 1 0 1" />
@@ -82,8 +85,10 @@
     </visual>
     <inertial>
+      <origin rpy="0 0 0" xyz="0 0 ${wheel_axle_offset + chassis_thickness/2}"/>
       <mass value="1.0"/>
       <inertia ixx="${(1/12)*(chassis_thickness**2 + chassis_width**2)}" iyy="${(1/12)*(chassis_thickness**2 + chassis_length**2)}" izz="${(1/12)*(chassis_length**2 + chassis_width**2)}" ixy="0" ixz="0" iyz="0"/>
     </inertial>
     <collision>
+      <origin rpy="0 0 0" xyz="0 0 ${wheel_axle_offset + chassis_thickness/2}"/>
       <geometry>
         <box size="${chassis_length} ${chassis_width} ${chassis_thickness}" />
@@ -92,5 +97,5 @@
   </link>
   <joint name="base_body" type="fixed">
-    <origin xyz="${base_shift} 0 ${wheel_axle_offset + chassis_thickness/2}" rpy="0 0 0" />
+    <origin xyz="${base_shift} 0 0" rpy="0 0 0" />
     <parent link="base_link"/>
     <child link="robot_body"/>
@@ -100,4 +105,4 @@
   <xacro:wheel_temp wheel_side="right" offset="-1"/>
   <!-- Caster Creation -->
-  <xacro:caster_temp caster_side="bottom" offset="-1"/>
+  <xacro:caster_temp caster_side="bottom"/>
 </robot>

Commit message: Finished Task G.005

File: nuturtle_description/urdf/diff_drive.urdf.xacro (robot description, xacro)
@@ -96,8 +96,18 @@
     </collision>
   </link>
-  <joint name="base_body" type="fixed">
+  <!-- Link body to base frame -->
+  <joint name="body_to_base" type="fixed">
     <origin xyz="${base_shift} 0 0" rpy="0 0 0" />
     <parent link="base_link"/>
     <child link="robot_body"/>
+  </joint>
+  <!-- The laser scanner -->
+  <link name="base_scan">
+    <origin rpy="0 0 0" xyz="$0 0 0"/>
+  </link>
+  <joint name="scan_to_base" type="fixed">
+    <origin xyz="0 0 ${chassis_thickness + wheel_axle_offset}" rpy="0 0 0" />
+    <parent link="base_link"/>
+    <child link="base_scan"/>
   </joint>
   <!-- Wheel Creation -->

File: nuturtle_gazebo/urdf/diff_drive.gazebo.xacro (robot description, xacro)
@@ -51,3 +51,35 @@
   <kd>100</kd>
 </gazebo>
+<gazebo reference="base_scan">
+  <material>Gazebo/FlatBlack</material>
+  <sensor type="ray" name="lds_lfcd_sensor">
+    <pose>0 0 0 0 0 0</pose>
+    <visualize>true</visualize>
+    <update_rate>5</update_rate>
+    <ray>
+      <scan>
+        <horizontal>
+          <samples>360</samples>
+          <resolution>1</resolution>
+          <min_angle>0.0</min_angle>
+          <max_angle>6.28319</max_angle>
+        </horizontal>
+      </scan>
+      <range>
+        <min>0.120</min>
+        <max>3.5</max>
+        <resolution>0.015</resolution>
+      </range>
+      <noise>
+        <type>gaussian</type>
+        <mean>0.0</mean>
+        <stddev>0.01</stddev>
+      </noise>
+    </ray>
+    <plugin name="gazebo_ros_lds_lfcd_controller" filename="libgazebo_ros_laser.so">
+      <topicName>scan</topicName>
+      <frameName>base_scan</frameName>
+    </plugin>
+  </sensor>
+</gazebo>
 </robot>

Commit message: Completed Task S.000 and S.001, Fully tested and tuned

File: nuturtle_description/urdf/diff_drive.urdf.xacro (robot description, xacro)
@@ -107,5 +107,5 @@
   </link>
   <joint name="scan_to_base" type="fixed">
-    <origin xyz="0 0 ${chassis_thickness + wheel_axle_offset}" rpy="0 0 0" />
+    <origin xyz="0.05 0 ${chassis_thickness + wheel_axle_offset}" rpy="0 0 0" /> <!-- added 2.5cm to prevent scan clipping robot corner in simulation -->
     <parent link="base_link"/>
     <child link="base_scan"/>
